File: bottomAcrylic/CZTKeyRev1AcrylicPlate.kicad_pcb (KiCad board)
At the start: 2 copper layers, 342.9 x 179.4 mm, 12 parts

Commit message: commit
Parts:
- moved PCB_BC1 195.0 mm to (180.2, -14.3)
- moved PCB_BL1 195.0 mm to (21.4, -14.3)
- moved PCB_BR1 195.0 mm to (338.1, -13.5)
- moved PCB_TC1 195.0 mm to (180.2, -102.4)
- moved PCB_TL1 195.0 mm to (10.3, -102.4)
- moved PCB_TR1 195.0 mm to (338.1, -117.5)
- moved PLATE_BC1 195.0 mm to (178.6, -130.2)
- moved PLATE_BL1 195.0 mm to (4.76, -131.0)
- moved PLATE_BR1 195.0 mm to (338.1, -131.0)
- moved PLATE_TC1 195.0 mm to (177.8, -174.6)
- moved PLATE_TL1 195.0 mm to (4.76, -174.6)
- moved PLATE_TR1 195.0 mm to (338.1, -174.6)
