File: pcb/CZTKeyRev1.kicad_pcb (KiCad board)
At the start: 2 copper layers, 342.9 x 174.6 mm, 363 parts, among them U1 proton_c

Commit message: Changed footprints
Parts:
- added MX_ALT_R1: MX-NoLED, MX_Only:MXOnly-1.5U-NoLED, F.Cu at (242.9, 180.2)
- MX_1, MX_10, MX_2, MX_3, MX_4, MX_5, MX_6, MX_7, MX_8, MX_9, MX_A1, MX_B1, MX_BR_L1, MX_BR_R1, MX_C1, MX_COMMA1, MX_D1, MX_DELETE1, MX_DOT1, MX_DOWN1, MX_E1, MX_EQUAL1, MX_ESC1, MX_F1, MX_F10, MX_F11, MX_F12, MX_F13, MX_F2, MX_F3, MX_F4, MX_F5, MX_F6, MX_F7, MX_F8, MX_F9, MX_G1, MX_H1, MX_I1, MX_INSERT1, MX_J1, MX_K1, MX_L1, MX_LEFT1, MX_M1, MX_MAC1, MX_MAC2, MX_MAC3, MX_MAC4, MX_MAC5, MX_MINUS1, MX_N1, MX_O1, MX_P1, MX_PGDWN1, MX_PGUP1, MX_PRTSC1, MX_Q1, MX_QUOTE1, MX_R1, MX_RIGHT1, MX_S1, MX_SEMIC1, MX_SLASH1, MX_T1, MX_TILDE1, MX_U1, MX_UP1, MX_V1, MX_W1, MX_X1, MX_Y1, MX_Z1: footprint MX_Alps_Hybrid:MX-1U-NoLED -> MX_Only:MXOnly-1U-NoLED
- MX_ALT_L1, MX_CTRL_L1, MX_WIN1: footprint MX_Alps_Hybrid:MX-1.25U-NoLED -> MX_Only:MXOnly-1.25U-NoLED
- MX_BACKSPACE1: footprint MX_Alps_Hybrid:MX-2U-NoLED -> MX_Only:MXOnly-2U-NoLED
- MX_BCKSLASH1, MX_CTRL_R1, MX_TAB1: footprint MX_Alps_Hybrid:MX-1.5U-NoLED -> MX_Only:MXOnly-1.5U-NoLED
- MX_CAPS1, MX_SHIFT_R1: footprint MX_Alps_Hybrid:MX-1.75U-NoLED -> MX_Only:MXOnly-1.75U-NoLED
- MX_ENTER1, MX_SHIFT_L1: footprint MX_Alps_Hybrid:MX-2.25U-NoLED -> MX_Only:MXOnly-2.25U-NoLED
- MX_SPACE1: footprint MX_Alps_Hybrid:MX-6.25U-NoLED -> MX_Only:MXOnly-6.25U-NoLED
Routing:
- net COL9: track 323.6 -> 318.0 mm
- net COL10: track 402.7 -> 399.4 mm
- net COL15: track 411.5 -> 408.3 mm
- net COL3: track 183.6 -> 180.4 mm
- net COL8: track 320.6 -> 317.5 mm
- net COL12: track 432.8 -> 429.6 mm
- net COL7: track 238.3 -> 235.5 mm
- net COL6: track 273.6 -> 270.8 mm
- net COL13: track 397.8 -> 395.1 mm
- net COL11: track 361.1 -> 358.7 mm
- net COL5: track 208.1 -> 206.0 mm
- net COL2: track 179.8 -> 178.8 mm
- net COL4: track 209.0 -> 208.3 mm
- net Net-(D87-Pad2): track 143.6 -> 143.0 mm
- net Net-(D84-Pad2): track 140.5 -> 139.9 mm
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Other:
- board text added: "Rev.1"
- board text removed: "Rev.0"

Commit message: commit
Parts:
- moved LED85 4.76 mm to (323.9, 190.2)
- moved LED75 4.76 mm to (323.9, 171.1)
- moved LED84 4.76 mm to (304.8, 190.1)
- moved LED86 4.76 mm to (342.9, 190.1)
- moved MX_DOWN1 4.76 mm to (323.9, 184.9)
- moved MX_LEFT1 4.76 mm to (304.8, 184.9)
- moved MX_RIGHT1 4.76 mm to (342.9, 184.9)
- moved MX_UP1 4.76 mm to (323.9, 165.9)
Routing:
- net EXT_5V: track 2471.3 -> 2513.5 mm, vias 4 -> 10
- net GND: track 2633.8 -> 2664.7 mm
- net Net-(D87-Pad2): track 143.0 -> 155.3 mm, vias 1 -> 2
- net Net-(LED81-Pad4): track 74.8 -> 86.1 mm
- net COL13: track 395.1 -> 401.6 mm
- net COL14: track 374.8 -> 379.6 mm
- net COL12: track 429.6 -> 434.4 mm
- net Net-(D86-Pad2): track 148.7 -> 153.4 mm
- net Net-(D85-Pad2): track 135.8 -> 140.5 mm
- net Net-(LED83-Pad4): track 28.8 -> 33.4 mm, vias 0 -> 2
- net Net-(D76-Pad2): track 105.2 -> 109.3 mm
- net Net-(LED74-Pad2): track 31.2 -> 35.1 mm, vias 0 -> 2
- net Net-(LED76-Pad2): track 32.0 -> 35.6 mm, vias 2 -> 4
- net Net-(EXT_IC1-Pad4): track 19.9 -> 22.5 mm
- net COL15: track 408.3 -> 406.3 mm
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Other:
- board size 342.9 x 174.6 mm -> 342.9 x 179.4 mm

Commit message: commit
Parts:
- D1, D10, D11, D12, D13, D14, D15, D16, D17, D18, D19, D2, D20, D21, D22, D23, D24, D25, D26, D27, D28, D29, D3, D30, D31, D32, D33, D34, D35, D36, D37, D38, D39, D4, D40, D41, D42, D43, D44, D45, D46, D47, D48, D49, D5, D50, D51, D52, D53, D54, D55, D56, D57, D58, D59, D6, D60, D61, D62, D63, D64, D65, D66, D67, D68, D69, D7, D70, D71, D72, D73, D74, D75, D76, D77, D78, D79, D8, D80, D81, D82, D83, D84, D85, D86, D87, D9: footprint Diode_THT:D_DO-35_SOD27_P5.08mm_Vertical_KathodeUp -> Diode_THT:D_DO-35_SOD27_P7.62mm_Horizontal
- moved D80 4.60 mm to (140.6, 45.2)
- moved DC84 4.32 mm to (313.1, 189.7)
- moved DC85 4.32 mm to (332.1, 189.7)
- moved D54 4.00 mm to (188.1, 43.7)
- moved D85 3.97 mm to (256.4, 59.5)
- moved D84 3.97 mm to (256.4, 45.3)
- moved D81 3.97 mm to (140.5, 58.7)
- moved D65 3.97 mm to (136.6, 44.5)
- moved D67 3.94 mm to (166.8, 44.5)
- moved BJ_LED5V1 3.91 mm to (26.2, 22.2)
- moved D58 3.70 mm to (188.1, 57.1)
- moved D38 3.59 mm to (184.2, 42.9)
- moved D68 3.37 mm to (166.7, 57.9)
- moved D66 3.37 mm to (136.5, 57.9)
- moved D50 3.37 mm to (132.6, 43.7)
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Routing:
- net EXT_5V: track 2513.5 -> 2672.0 mm, vias 10 -> 4
- net GND: track 2664.7 -> 2745.6 mm, vias 14 -> 10
- net COL10: track 399.4 -> 329.5 mm
- net COL15: track 406.3 -> 462.1 mm, vias 0 -> 2
- net COL12: track 434.4 -> 384.6 mm, vias 2 -> 1
- net COL8: track 317.5 -> 269.8 mm, vias 2 -> 4
- net COL4: track 208.3 -> 165.4 mm
- net Net-(D39-Pad2): track 121.2 -> 86.1 mm
- net Net-(D41-Pad2): track 141.0 -> 175.7 mm, vias 2 -> 1
- net Net-(D57-Pad2): track 167.3 -> 197.3 mm, vias 2 -> 1
- net Net-(D62-Pad2): track 136.3 -> 108.6 mm
- net Net-(D77-Pad2): track 151.5 -> 126.2 mm
- net Net-(D83-Pad2): track 163.8 -> 139.2 mm, vias 1 -> 0
- net ROW5: track 357.5 -> 381.7 mm
- net Net-(D67-Pad2): track 144.6 -> 120.6 mm
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